Commit message: First upload

File: docker_ws/arm_ws/src/mycobot_ros2/mycobot_gazebo/urdf/ros2_control/classic_gazebo/mycobot_280.urdf.xacro (robot description, xacro)
@@ -388,5 +388,5 @@
 		<child link="link2"/>
 		<origin xyz= "0 0 0.13156" rpy = "0 0 ${pi/2}"/>
-        <dynamics damping="12.0" friction="6.0"/>
+        <dynamics damping="1000.0" friction="100.0"/>
 	</joint>
 	<joint name="link2_to_link3" type="revolute">
@@ -396,5 +396,5 @@
 		<child link="link3"/>
 		<origin xyz= "0 0 -0.001" rpy = "0 ${pi/2} ${-pi/2}"/>
-        <dynamics damping="12.0" friction="6.0"/>
+        <dynamics damping="1000.0" friction="100.0"/>
 	</joint>
 	<joint name="link3_to_link4" type="revolute">
@@ -404,5 +404,5 @@
 		<child link="link4"/>
 		<origin xyz= "-0.1104 0 0   " rpy = "0 0 0"/>
-        <dynamics damping="12.0" friction="6.0"/>
+        <dynamics damping="1000.0" friction="100.0"/>
 	</joint>
 	<joint name="link4_to_link5" type="revolute">
@@ -412,5 +412,5 @@
 		<child link="link5"/>
 		<origin xyz= "-0.096 0 0.06062" rpy = "0 0 ${-pi/2}"/>
-        <dynamics damping="12.0" friction="6.0"/>
+        <dynamics damping="1000.0" friction="100.0"/>
 	</joint>
 	<joint name="link5_to_link6" type="revolute">
@@ -420,5 +420,5 @@
 		<child link="link6"/>
 		<origin xyz= "0 -0.07318 0" rpy = "${pi/2} ${-pi/2} 0"/>
-        <dynamics damping="7.0" friction="4.0"/>
+        <dynamics damping="1000.0" friction="100"/>
 	</joint>
 	<joint name="link6_to_link6flange" type="revolute">
@@ -428,5 +428,5 @@
 		<child link="link6_flange"/>
 		<origin xyz= "0 0.0456 0" rpy = "${-pi/2} 0 0"/>
-        <dynamics damping="3.0" friction="3.0"/>
+        <dynamics damping="1000.0" friction="100.0"/>
 	</joint>
 	<joint name="link6flange_to_gripper_base" type="fixed">
@@ -441,5 +441,5 @@
 		<child link="gripper_left3"/>
 		<origin xyz= "-0.012 0.005 0" rpy = "0 0 0"/>
-        <dynamics damping="2.0" friction="4.0"/>
+        <dynamics damping="1000.0" friction="100.0"/>
 	</joint>
 	<joint name="gripper_base_to_gripper_left2" type="revolute">
@@ -450,5 +450,5 @@
 		<origin xyz= "-0.005 0.027 0" rpy = "0 0 0"/>
 		<mimic joint="gripper_controller" multiplier="1.0" offset="0" />
-        <dynamics damping="2.0" friction="4.0"/>
+        <dynamics damping="1000.0" friction="100.0"/>
 	</joint>
 	<joint name="gripper_left3_to_gripper_left1" type="revolute">
@@ -459,5 +459,5 @@
 		<origin xyz= "-0.027 0.016 0" rpy = "0 0 0"/>
 		<mimic joint="gripper_controller" multiplier="-1.0" offset="0" />
-        <dynamics damping="2.0" friction="4.0"/>
+        <dynamics damping="1000.0" friction="100.0"/>
 	</joint>
 	<joint name="gripper_base_to_gripper_right3" type="revolute">
@@ -468,5 +468,5 @@
 		<origin xyz= "0.012 0.005 0" rpy = "0 0 0"/>
 		<mimic joint="gripper_controller" multiplier="-1.0" offset="0" />
-        <dynamics damping="2.0" friction="4.0"/>
+        <dynamics damping="1000.0" friction="100.0"/>
 	</joint>
 	<joint name="gripper_base_to_gripper_right2" type="revolute">
@@ -477,5 +477,5 @@
 		<origin xyz= "0.005 0.027 0" rpy = "0 0 0"/>
 		<mimic joint="gripper_controller" multiplier="-1.0" offset="0" />
-        <dynamics damping="2.0" friction="4.0"/>
+        <dynamics damping="1000.0" friction="100.0"/>
 	</joint>
 	<joint name="gripper_right3_to_gripper_right1" type="revolute">
@@ -486,5 +486,5 @@
 		<origin xyz= "0.027 0.016 0" rpy = "0 0 0"/>
 		<mimic joint="gripper_controller" multiplier="1.0" offset="0" />
-        <dynamics damping="2.0" friction="4.0"/>
+        <dynamics damping="1000.0" friction="100.0"/>
 	</joint>
     <xacro:default_transmission joint_name="link1_to_link2"/>

File: docker_ws/arm_ws/src/mycobot_ros2/mycobot_gazebo/urdf/ros2_control/classic_gazebo/mycobot_280_classic_gazebo.xacro (robot description, xacro)
@@ -1,11 +1,4 @@
 <?xml version="1.0" ?>
 <robot xmlns:xacro="http://wiki.ros.org/xacro" name="mycobot_280">
-    <!-- The Gazebo plugin for ros2_control -->
-    <gazebo>
-        <plugin filename="libgazebo_ros2_control.so" name="gazebo_ros2_control">
-            <robot_param>robot_description</robot_param>
-            <robot_param_node>robot_state_publisher</robot_param_node>
-            <parameters>$(find mycobot_gazebo)/config/mycobot_280_controllers.yaml</parameters>
-        </plugin>
-    </gazebo>
+    <!-- NO gazebo_ros2_control plugin - using direct PID control instead -->
 </robot>
