Commit message: Added gazebo ros2 control plugin to the urdf i am using

File: docker_ws/arm_ws/src/mycobot_ros2/mycobot_gazebo/urdf/ros2_control/classic_gazebo/mycobot_280_gazebo_classic.urdf.xacro (robot description, xacro)
@@ -1,52 +1,53 @@
 <?xml version="1.0" ?>
 <robot xmlns:xacro="http://wiki.ros.org/xacro" name="mycobot_280">
-  <!-- Disable gravity for all links -->
+    <!-- Disable gravity -->
     <gazebo>
         <gravity>0 0 0</gravity>
     </gazebo>
-    <!-- Include the complete robot model from gazebo directory -->
+    <!-- Include the complete robot model -->
     <xacro:include filename="$(find mycobot_gazebo)/urdf/ros2_control/gazebo/mycobot_280.urdf.xacro"/>
-    <!-- Gazebo Joint State Publisher Plugin -->
+    <!-- ros2_control hardware interface -->
+    <ros2_control name="GazeboSystem" type="system">
+        <hardware>
+            <plugin>gazebo_ros2_control/GazeboSystem</plugin>
+        </hardware>
+        <joint name="link1_to_link2">
+            <command_interface name="position"/>
+            <state_interface name="position"/>
+            <state_interface name="velocity"/>
+        </joint>
+        <joint name="link2_to_link3">
+            <command_interface name="position"/>
+            <state_interface name="position"/>
+            <state_interface name="velocity"/>
+        </joint>
+        <joint name="link3_to_link4">
+            <command_interface name="position"/>
+            <state_interface name="position"/>
+            <state_interface name="velocity"/>
+        </joint>
+        <joint name="link4_to_link5">
+            <command_interface name="position"/>
+            <state_interface name="position"/>
+            <state_interface name="velocity"/>
+        </joint>
+        <joint name="link5_to_link6">
+            <command_interface name="position"/>
+            <state_interface name="position"/>
+            <state_interface name="velocity"/>
+        </joint>
+        <joint name="link6_to_link6flange">
+            <command_interface name="position"/>
+            <state_interface name="position"/>
+            <state_interface name="velocity"/>
+        </joint>
+    </ros2_control>
+    <!-- Gazebo ros2_control plugin -->
     <gazebo>
-        <plugin name="gazebo_ros_joint_state_publisher" filename="libgazebo_ros_joint_state_publisher.so">
-            <update_rate>100</update_rate>
-            <joint_name>link1_to_link2</joint_name>
-            <joint_name>link2_to_link3</joint_name>
-            <joint_name>link3_to_link4</joint_name>
-            <joint_name>link4_to_link5</joint_name>
-            <joint_name>link5_to_link6</joint_name>
-            <joint_name>link6_to_link6flange</joint_name>
+        <plugin filename="libgazebo_ros2_control.so" name="gazebo_ros2_control">
+            <robot_param>robot_description</robot_param>
+            <robot_param_node>robot_state_publisher</robot_param_node>
+            <parameters>$(find mycobot_moveit_config)/config/ros2_controllers.yaml</parameters>
         </plugin>
     </gazebo>
-    <!-- Gazebo Position Controllers for each joint -->
-    <gazebo>
-        <plugin name="gazebo_ros_joint_pose_trajectory" filename="libgazebo_ros_joint_pose_trajectory.so">
-            <update_rate>100</update_rate>
-            <joint_name>link1_to_link2</joint_name>
-            <joint_name>link2_to_link3</joint_name>
-            <joint_name>link3_to_link4</joint_name>
-            <joint_name>link4_to_link5</joint_name>
-            <joint_name>link5_to_link6</joint_name>
-            <joint_name>link6_to_link6flange</joint_name>
-        </plugin>
-    </gazebo>
-    <!-- Add PID gains for each joint to fight gravity and hold positions -->
-    <gazebo reference="link1_to_link2">
-        <implicitSpringDamper>true</implicitSpringDamper>
-    </gazebo>
-    <gazebo reference="link2_to_link3">
-        <implicitSpringDamper>true</implicitSpringDamper>
-    </gazebo>
-    <gazebo reference="link3_to_link4">
-        <implicitSpringDamper>true</implicitSpringDamper>
-    </gazebo>
-    <gazebo reference="link4_to_link5">
-        <implicitSpringDamper>true</implicitSpringDamper>
-    </gazebo>
-    <gazebo reference="link5_to_link6">
-        <implicitSpringDamper>true</implicitSpringDamper>
-    </gazebo>
-    <gazebo reference="link6_to_link6flange">
-        <implicitSpringDamper>true</implicitSpringDamper>
-    </gazebo>
 </robot>
